File: Minus_X_Panel_X3.kicad_sch (KiCad schematic)
At the start: 0 parts

Commit message: footprint of the Panel is modified with tracking
Parts:
- added D1, D2, D3: CUHS20S30,H3F, Custom-Footprints:CUHS20S30,H3F, symbol Custom-Symbols:CUHS20S30,H3F
- added S1, S3: solar_cell_B, Custom-Footprints:solar_cell_B, symbol Custom-Symbols:solar_cell_B
- added S2, S4: Solar_cell_C, Custom-Footprints:solar_cell_C, symbol Custom-Symbols:Solar_cell_C
- added U$1: 2PIN_FEMALE, Custom-Footprints:FSR-41057-02-F, symbol Custom-Symbols:2PIN_FEMALE
- added U$2: 2PIN_MALE, Custom-Footprints:PSR-410253-02-M, symbol Custom-Symbols:2PIN_MALE
- added U$3: 3PIN_FEMALE_-XC3PIN_MALE, Custom-Footprints:FSR-41057-03-F, symbol Custom-Symbols:3PIN_FEMALE_-XC3PIN_MALE
- added U$4: 3PIN_MALE3PIN_MALE, Custom-Footprints:PSR-410253-03-M, symbol Custom-Symbols:3PIN_MALE3PIN_MALE
Connections:
- new net: D3.2 (A), S4.GND, U$4.3P*
- new net: D1.1 (K), U$1.1PWR, U$1.2PWR, U$2.1PWR, U$2.2PWR
- new net +V3A: D2.1 (K), S2.+V, S3.GND
- new net +V3B: S1.GND, S3.+V
- new net +V3C: D1.2 (A), S1.+V
- new net +V3D: D3.1 (K), S4.+V, U$3.3P*
- new net GND: D2.2 (A), S2.GND, U$3.1GND, U$3.GND, U$4.1GND, U$4.GND
